File: STM32F103C8T6.kicad_sch (KiCad schematic)
At the start: 29 parts, among them SW1 SW_Push, SW2 SW_Push, U1 STM32F103C8T6, U2 AMS1117-3.3

Commit message: Update to KiCAD 7.0
Parts:
- removed CH1, CH2: Conn_01x20_Male, Connector_PinHeader_2.54mm:PinHeader_1x20_P2.54mm_Vertical, symbol Connector:Conn_01x20_Male
- removed R3: 10KΩ, Resistor_SMD:R_0402_1005Metric, symbol Device:R
- removed UART1: Conn_01x06_Male, Connector_PinHeader_2.54mm:PinHeader_1x06_P2.54mm_Horizontal, symbol Connector:Conn_01x06_Male
- added CH1, CH2: Conn_01x20, Connector_PinHeader_2.54mm:PinHeader_1x20_P2.54mm_Vertical, symbol Connector_Generic:Conn_01x20
- added H3, H4: MountingHole, MountingHole:MountingHole_2.2mm_M2, symbol Mechanical:MountingHole
- added UART1: Conn_01x06, Connector_PinHeader_2.54mm:PinHeader_1x06_P2.54mm_Horizontal, symbol Connector_Generic:Conn_01x06
- C11: value 10μF -> 1μF; footprint Capacitor_SMD:C_0603_1608Metric -> Capacitor_SMD:C_0402_1005Metric; LCSC C19702 -> C52923
- C12: value 22μF -> 100μF; footprint Capacitor_SMD:C_0603_1608Metric -> Capacitor_SMD:C_1206_3216Metric; LCSC C59461 -> C15008
- U1: LCSC (none) -> C8734
Connections:
- net +3.3V: now also CH1.18 (Pin_18)
- net +5V: now also CH1.20 (Pin_20), UART1.4 (Pin_4)
- net GND: now also CH1.19 (Pin_19), CH2.20 (Pin_20), UART1.5 (Pin_5), UART1.6 (Pin_6)
- net NRST: now also CH1.17 (Pin_17)
- net PA0: now also CH1.4 (Pin_4)
- net PA1: now also CH1.5 (Pin_5)
- net PA10: now also CH2.13 (Pin_13), UART1.3 (Pin_3)
- net PA11: now also CH2.12 (Pin_12)
- net PA12: now also CH2.11 (Pin_11)
- net PA13: now also CH2.10 (Pin_10)
- net PA14: now also CH2.9 (Pin_9)
- net PA15: now also CH2.8 (Pin_8)
- net PA2: now also CH1.6 (Pin_6)
- net PA3: now also CH1.7 (Pin_7)
- net PA4: now also CH1.8 (Pin_8)
- net PA5: now also CH1.9 (Pin_9)
- net PA6: now also CH1.10 (Pin_10)
- net PA7: now also CH1.11 (Pin_11)
- net PA8: now also CH2.15 (Pin_15)
- net PA9: now also CH2.14 (Pin_14), UART1.2 (Pin_2)
- net PB0: now also CH1.12 (Pin_12)
- net PB1: now also CH1.13 (Pin_13)
- net PB10: now also CH1.15 (Pin_15)
- net PB11: now also CH1.16 (Pin_16)
- net PB12: now also CH2.19 (Pin_19)
- net PB13: now also CH2.18 (Pin_18)
- net PB14: now also CH2.17 (Pin_17)
- net PB15: now also CH2.16 (Pin_16)
- net PB2: now also CH1.14 (Pin_14)
- net PB3: now also CH2.7 (Pin_7)
- net PB4: now also CH2.6 (Pin_6)
- net PB5: now also CH2.5 (Pin_5)
- net PB6: now also CH2.4 (Pin_4)
- net PB7: now also CH2.3 (Pin_3)
- net PB8: now also CH2.2 (Pin_2)
- net PB9: now also CH2.1 (Pin_1)
- net PC13: now also CH1.1 (Pin_1)
- net PC14: now also CH1.2 (Pin_2)
- net PC15: now also CH1.3 (Pin_3)
Other:
- moved on the sheet: H1, H2

Commit message: Add files via upload
Parts:
- removed H1, H2, H3, H4: MountingHole, MountingHole:MountingHole_2.2mm_M2, symbol Mechanical:MountingHole
Changed lines of the file:
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@@
-    )
-  )
-  (symbol (lib_id "Mechanical:MountingHole") (at 210.82 43.18 0) (unit 1)
-    (in_bom yes) (on_board yes) (dnp no) (fields_autoplaced)
-    (property "Reference" "H2" (at 213.36 41.9099 0)
-      (effects (font (size 1.27 1.27)) (justify left))
-    )
-    (property "Value" "MountingHole" (at 213.36 44.4499 0)
-      (effects (font (size 1.27 1.27)) (justify left))
-    )
-    (property "Footprint" "MountingHole:MountingHole_2.2mm_M2" (at 210.82 43.18 0)
-      (effects (font (size 1.27 1.27)) hide)
-    )
-    (property "Datasheet" "~" (at 210.82 43.18 0)
-      (effects (font (size 1.27 1.27)) hide)
-    )
-    (instances
-      (project "STM32F103C8T6"
-        (path "/978e1817-ddd6-4f04-b9a6-ae7fae5b1d1d"
-          (reference "H2") (unit 1)
-        )
-      )
     )
   )
@@
     )
   )
-  (symbol (lib_id "Mechanical:MountingHole") (at 232.41 36.83 0) (unit 1)
-    (in_bom yes) (on_board yes) (dnp no) (fields_autoplaced)
-    (property "Reference" "H3" (at 234.95 35.5599 0)
-      (effects (font (size 1.27 1.27)) (justify left))
-    )
-    (property "Value" "MountingHole" (at 234.95 38.0999 0)
-      (effects (font (size 1.27 1.27)) (justify left))
-    )
-    (property "Footprint" "MountingHole:MountingHole_2.2mm_M2" (at 232.41 36.83 0)
-      (effects (font (size 1.27 1.27)) hide)
-    )
-    (property "Datasheet" "~" (at 232.41 36.83 0)
-      (effects (font (size 1.27 1.27)) hide)
-    )
-    (instances
-      (project "STM32F103C8T6"
-        (path "/978e1817-ddd6-4f04-b9a6-ae7fae5b1d1d"
-          (reference "H3") (unit 1)
-        )
-      )
-    )
-  )
   (symbol (lib_id "power:PWR_FLAG") (at 106.68 35.56 0) (unit 1)
     (in_bom yes) (on_board yes) (dnp no)
@@
     )
   )
-  (symbol (lib_id "Mechanical:MountingHole") (at 232.41 43.18 0) (unit 1)
-    (in_bom yes) (on_board yes) (dnp no) (fields_autoplaced)
-    (property "Reference" "H4" (at 234.95 41.9099 0)
-      (effects (font (size 1.27 1.27)) (justify left))
-    )
-    (property "Value" "MountingHole" (at 234.95 44.4499 0)
-      (effects (font (size 1.27 1.27)) (justify left))
-    )
-    (property "Footprint" "MountingHole:MountingHole_2.2mm_M2" (at 232.41 43.18 0)
-      (effects (font (size 1.27 1.27)) hide)
-    )
-    (property "Datasheet" "~" (at 232.41 43.18 0)
-      (effects (font (size 1.27 1.27)) hide)
-    )
-    (instances
-      (project "STM32F103C8T6"
-        (path "/978e1817-ddd6-4f04-b9a6-ae7fae5b1d1d"
-          (reference "H4") (unit 1)
-        )
-      )
-    )
-  )
   (symbol (lib_id "Device:R") (at 173.99 38.1 90) (unit 1)
     (in_bom yes) (on_board yes) (dnp no) (fields_autoplaced)
@@
         )
       )
-    )
-  )
-  (symbol (lib_id "Mechanical:MountingHole") (at 210.82 36.83 0) (unit 1)
-    (in_bom yes) (on_board yes) (dnp no) (fields_autoplaced)
-    (property "Reference" "H1" (at 213.36 35.5599 0)
-      (effects (font (size 1.27 1.27)) (justify left))
-    )
-    (property "Value" "MountingHole" (at 213.36 38.0999 0)
-      (effects (font (size 1.27 1.27)) (justify left))
-    )
-    (property "Footprint" "MountingHole:MountingHole_2.2mm_M2" (at 210.82 36.83 0)
-      (effects (font (size 1.27 1.27)) hide)
-    )
-    (property "Datasheet" "~" (at 210.82 36.83 0)
-      (effects (font (size 1.27 1.27)) hide)
-    )
-    (instances
-      (project "STM32F103C8T6"
-        (path "/978e1817-ddd6-4f04-b9a6-ae7fae5b1d1d"
-          (reference "H1") (unit 1)
-        )
-      )
