File: STM32F1-DevBoard.kicad_sch (KiCad schematic)
At the start: 32 parts, among them SW1 SW_Push, SW2 SW_Push, U1 STM32F103C8T6, U2 AMS1117-3.3, U3 W25Q32JVSS

Commit message: Add files via upload
Parts:
- LED1: renamed from D1; value 19-217/BHC-ZL1M2RY/3T -> 19-217/GHC-YR1S2/3T; LCSC C72041 -> C72043
- LED2: renamed from D2; value 19-217/GHC-YR1S2/3T -> KT-0603R; LCSC C72043 -> C2286
Changed lines of the file:
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@@
     (stroke (width 0) (type default))
   )
-  (wire (pts (xy 115.57 39.37) (xy 118.11 39.37))
+  (wire (pts (xy 115.57 39.37) (xy 120.65 39.37))
     (stroke (width 0) (type default))
   )
@@
     (stroke (width 0) (type default))
   )
-  (wire (pts (xy 92.71 39.37) (xy 95.25 39.37))
+  (wire (pts (xy 90.17 39.37) (xy 95.25 39.37))
     (stroke (width 0) (type default))
   )
@@
     )
   )
-  (symbol (lib_id "power:+5V") (at 92.71 39.37 90) (unit 1)
+  (symbol (lib_id "power:+5V") (at 90.17 39.37 90) (unit 1)
     (in_bom yes) (on_board yes) (dnp no) (fields_autoplaced)
-    (property "Reference" "#PWR0117" (at 96.52 39.37 0)
-      (effects (font (size 1.27 1.27)) hide)
-    )
-    (property "Value" "+5V" (at 88.9 39.3699 90)
+    (property "Reference" "#PWR0117" (at 93.98 39.37 0)
+      (effects (font (size 1.27 1.27)) hide)
+    )
+    (property "Value" "+5V" (at 86.36 39.3699 90)
       (effects (font (size 1.27 1.27)) (justify left))
     )
-    (property "Footprint" "" (at 92.71 39.37 0)
-      (effects (font (size 1.27 1.27)) hide)
-    )
-    (property "Datasheet" "" (at 92.71 39.37 0)
+    (property "Footprint" "" (at 90.17 39.37 0)
+      (effects (font (size 1.27 1.27)) hide)
+    )
+    (property "Datasheet" "" (at 90.17 39.37 0)
       (effects (font (size 1.27 1.27)) hide)
     )
@@
   (symbol (lib_id "Device:LED") (at 154.94 41.91 180) (unit 1)
     (in_bom yes) (on_board yes) (dnp no)
-    (property "Reference" "D1" (at 156.21 29.21 0)
-      (effects (font (size 1.27 1.27)))
-    )
-    (property "Value" "19-217/BHC-ZL1M2RY/3T" (at 156.21 31.75 0)
-      (effects (font (size 1.27 1.27)))
+    (property "Reference" "LED1" (at 158.75 35.56 0)
+      (effects (font (size 1.27 1.27)) (justify left))
+    )
+    (property "Value" "19-217/GHC-YR1S2/3T" (at 158.75 38.1 0)
+      (effects (font (size 1.27 1.27)) (justify left))
     )
     (property "Footprint" "LED_SMD:LED_0603_1608Metric" (at 154.94 41.91 0)
       (effects (font (size 1.27 1.27)) hide)
     )
-    (property "Datasheet" "https://datasheet.lcsc.com/lcsc/1811101510_Everlight-Elec-19-217-BHC-ZL1M2RY-3T_C72041.pdf" (at 154.94 41.91 0)
-      (effects (font (size 1.27 1.27)) hide)
-    )
-    (property "LCSC" "C72041" (at 154.94 41.91 0)
+    (property "Datasheet" "https://datasheet.lcsc.com/lcsc/1811101510_Everlight-Elec-19-217-GHC-YR1S2-3T_C72043.pdf" (at 154.94 41.91 0)
+      (effects (font (size 1.27 1.27)) hide)
+    )
+    (property "LCSC" "C72043" (at 154.94 41.91 0)
       (effects (font (size 1.27 1.27)) hide)
     )
@@
       (project "STM32F1-DevBoard"
         (path "/978e1817-ddd6-4f04-b9a6-ae7fae5b1d1d"
-          (reference "D1") (unit 1)
+          (reference "LED1") (unit 1)
         )
       )
@@
   (symbol (lib_id "Device:LED") (at 154.94 46.99 180) (unit 1)
     (in_bom yes) (on_board yes) (dnp no)
-    (property "Reference" "D2" (at 156.21 58.42 0)
-      (effects (font (size 1.27 1.27)))
-    )
-    (property "Value" "19-217/GHC-YR1S2/3T" (at 156.21 55.88 0)
-      (effects (font (size 1.27 1.27)))
+    (property "Reference" "LED2" (at 158.75 53.34 0)
+      (effects (font (size 1.27 1.27)) (justify left))
+    )
+    (property "Value" "KT-0603R" (at 158.75 50.8 0)
+      (effects (font (size 1.27 1.27)) (justify left))
     )
     (property "Footprint" "LED_SMD:LED_0603_1608Metric" (at 154.94 46.99 0)
       (effects (font (size 1.27 1.27)) hide)
     )
-    (property "Datasheet" "https://datasheet.lcsc.com/lcsc/1811101510_Everlight-Elec-19-217-GHC-YR1S2-3T_C72043.pdf" (at 154.94 46.99 0)
-      (effects (font (size 1.27 1.27)) hide)
-    )
-    (property "LCSC" "C72043" (at 154.94 46.99 0)
+    (property "Datasheet" "https://datasheet.lcsc.com/lcsc/1810231112_Hubei-KENTO-Elec-KT-0603R_C2286.pdf" (at 154.94 46.99 0)
+      (effects (font (size 1.27 1.27)) hide)
+    )
+    (property "LCSC" "C2286" (at 154.94 46.99 0)
       (effects (font (size 1.27 1.27)) hide)
     )
@@
       (project "STM32F1-DevBoard"
         (path "/978e1817-ddd6-4f04-b9a6-ae7fae5b1d1d"
-          (reference "D2") (unit 1)
+          (reference "LED2") (unit 1)
         )
       )
@@
     )
   )
-  (symbol (lib_id "power:+3.3V") (at 118.11 39.37 270) (unit 1)
+  (symbol (lib_id "power:+3.3V") (at 120.65 39.37 270) (unit 1)
     (in_bom yes) (on_board yes) (dnp no) (fields_autoplaced)
-    (property "Reference" "#PWR0118" (at 114.3 39.37 0)
-      (effects (font (size 1.27 1.27)) hide)
-    )
-    (property "Value" "+3.3V" (at 121.92 39.3699 90)
+    (property "Reference" "#PWR0118" (at 116.84 39.37 0)
+      (effects (font (size 1.27 1.27)) hide)
+    )
+    (property "Value" "+3.3V" (at 124.46 39.3699 90)
       (effects (font (size 1.27 1.27)) (justify left))
     )
-    (property "Footprint" "" (at 118.11 39.37 0)
-      (effects (font (size 1.27 1.27)) hide)
-    )
-    (property "Datasheet" "" (at 118.11 39.37 0)
-      (effects (font (size 1.27 1.27)) hide)
-    )
+    (property "Footprint" "" (at 120.65 39.37 0)
+      (effects (font (size 1.27 1.27)) hide)
+    )
+    (property "Datasheet" "" (at 120.65 39.37 0)
+      (effects (font (size 1.27 1.27)) hide)
+    )

Commit message: Add files via upload
Parts:
- removed D4: 1N5819WS, Diode_SMD:D_SOD-323, symbol Diode:1N5819WS
- removed UART1: Conn_01x06, Connector_PinHeader_2.54mm:PinHeader_1x06_P2.54mm_Horizontal, symbol Connector_Generic:Conn_01x06
- added D1: 1N5819WS, Diode_SMD:D_SOD-323, symbol Diode:1N5819WS
- added H1, H2, H3, H4: MountingHole, MountingHole:MountingHole_2.2mm_M2, symbol Mechanical:MountingHole
- added J1: USB_C_Receptacle_USB2.0, Connector_USB:USB_C_Receptacle_XKB_U262-16XN-4BVC11, symbol Connector:USB_C_Receptacle_USB2.0
- added R3, R6: 5.1kΩ, Resistor_SMD:R_0402_1005Metric, symbol Device:R
- added R7: 1.5kΩ, Resistor_SMD:R_0402_1005Metric, symbol Device:R
- C1, C2: value 15pF -> 10pF; LCSC C1548 -> C32949
- C11: value 1μF -> 10uF; LCSC C52923 -> C15525
- C12: value 100μF -> 10uF; footprint Capacitor_SMD:C_1206_3216Metric -> Capacitor_SMD:C_0402_1005Metric; LCSC C15008 -> C15525
- C3, C4: value 30pF -> 20pF; LCSC C1570 -> C1554
- C6: footprint Capacitor_SMD:C_0603_1608Metric -> Capacitor_SMD:C_0603_1608Metric_Pad1.08x0.95mm_HandSolder; LCSC (none) -> C14663
- R1, R2, R4, R5: value 10KΩ -> 10kΩ
- XTAL2: footprint Crystal:Crystal_SMD_HC49-SD -> Crystal:Crystal_SMD_5032-2Pin_5.0x3.2mm; LCSC C12674 -> C115962
Connections:
- net +3.3V: now also R7.1
- net +5V: no longer C11.1, U2.3 (VI)
- net GND: now also C2.2, C4.2, J1.A1 (GND), J1.A12 (GND), J1.B1 (GND), J1.B12 (GND), J1.S1 (SHIELD), R3.1, R6.1; no longer C2.1, C4.1
- net PA11: now also J1.A7 (D-), J1.B7 (D-)
- net PA12: now also J1.A6 (D+), J1.B6 (D+), R7.2
- net PC15: now also C2.1; no longer C2.2
- net PD1: now also C4.1; no longer C4.2
- new net: J1.B5 (CC2), R6.2
- new net: J1.A5 (CC1), R3.2
- new net VBUS: D1.2 (A), J1.A4 (VBUS), J1.A9 (VBUS), J1.B4 (VBUS), J1.B9 (VBUS)
- new net VCC: C11.1, D1.1 (K), U2.3 (VI)
- no-connect marks 1 -> 2
Other:
- title: STM32F103C8T6 -> STM32F1-DevBoard
- moved on the sheet: C1, C10, C11, C12, C13, C3, C5, C6, C7, C8, C9, CH1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

Commit message: Add files via upload
Other:
- moved on the sheet: C1, C10, C11, C12, C13, C2, C3, C4, C5, C6, C7, C8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

Commit message: Add files via upload
Connections:
- net +5V is gone; now on net VBUS: CH1.20 (Pin_20)
Changed lines of the file:
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@@
+    )
+  )
+  (symbol (lib_id "power:VBUS") (at 193.04 147.32 90) (unit 1)
+    (in_bom yes) (on_board yes) (dnp no) (fields_autoplaced)
+    (property "Reference" "#PWR04" (at 196.85 147.32 0)
+      (effects (font (size 1.27 1.27)) hide)
+    )
+    (property "Value" "VBUS" (at 189.23 147.32 90)
+      (effects (font (size 1.27 1.27)) (justify left))
+    )
+    (property "Footprint" "" (at 193.04 147.32 0)
+      (effects (font (size 1.27 1.27)) hide)
+    )
+    (property "Datasheet" "" (at 193.04 147.32 0)
+      (effects (font (size 1.27 1.27)) hide)
+    )
+    (pin "1")
+    (instances
+      (project "STM32F1-DevBoard"
+        (path "/978e1817-ddd6-4f04-b9a6-ae7fae5b1d1d"
+          (reference "#PWR04") (unit 1)
+        )
+      )
     )
   )
@@
         )
       )
-    )
-  )
-  (symbol (lib_id "power:+5V") (at 193.04 147.32 90) (unit 1)
-    (in_bom yes) (on_board yes) (dnp no)
-    (property "Reference" "#PWR04" (at 196.85 147.32 0)
-      (effects (font (size 1.27 1.27)) hide)
-    )
-    (property "Value" "+5V" (at 187.96 147.32 90)
-      (effects (font (size 1.27 1.27)))
-    )
-    (property "Footprint" "" (at 193.04 147.32 0)
-      (effects (font (size 1.27 1.27)) hide)
-    )
-    (property "Datasheet" "" (at 193.04 147.32 0)
-      (effects (font (size 1.27 1.27)) hide)
-    )
-    (pin "1")
-    (instances
-      (project "STM32F1-DevBoard"
-        (path "/978e1817-ddd6-4f04-b9a6-ae7fae5b1d1d"
-          (reference "#PWR04") (unit 1)
-        )
-      )

Commit message: Add files via upload
Other:
- moved on the sheet: C10, C7, C8, C9, CH1, CH2, FB1, R1, U1

Commit message: Add files via upload
Parts:
- XTAL2: JLCPCB Rotation Offset -180 -> 0
Changed lines of the file:
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@@
       (effects (font (size 1.27 1.27)) hide)
     )
-    (property "JLCPCB Rotation Offset" "-180" (at 107.95 143.51 90)
+    (property "JLCPCB Rotation Offset" "0" (at 107.95 143.51 90)
       (effects (font (size 1.27 1.27)) hide)
     )

Commit message: Add files via upload
Connections:
- net VBUS: no longer CH1.20 (Pin_20)
- net VCC: now also CH1.20 (Pin_20)
Changed lines of the file:
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@@
-    )
-  )
-  (symbol (lib_id "power:VBUS") (at 193.04 148.59 90) (unit 1)
-    (in_bom yes) (on_board yes) (dnp no) (fields_autoplaced)
-    (property "Reference" "#PWR04" (at 196.85 148.59 0)
-      (effects (font (size 1.27 1.27)) hide)
-    )
-    (property "Value" "VBUS" (at 189.23 148.59 90)
-      (effects (font (size 1.27 1.27)) (justify left))
-    )
-    (property "Footprint" "" (at 193.04 148.59 0)
-      (effects (font (size 1.27 1.27)) hide)
-    )
-    (property "Datasheet" "" (at 193.04 148.59 0)
-      (effects (font (size 1.27 1.27)) hide)
-    )
-    (pin "1")
-    (instances
-      (project "STM32F1-DevBoard"
-        (path "/978e1817-ddd6-4f04-b9a6-ae7fae5b1d1d"
-          (reference "#PWR04") (unit 1)
-        )
-      )
     )
   )
@@
         )
       )
+    )
+  )
+  (symbol (lib_id "power:VCC") (at 193.04 148.59 90) (unit 1)
+    (in_bom yes) (on_board yes) (dnp no) (fields_autoplaced)
+    (property "Reference" "#PWR04" (at 196.85 148.59 0)
+      (effects (font (size 1.27 1.27)) hide)
+    )
+    (property "Value" "VCC" (at 189.23 148.59 90)
+      (effects (font (size 1.27 1.27)) (justify left))
+    )
+    (property "Footprint" "" (at 193.04 148.59 0)
+      (effects (font (size 1.27 1.27)) hide)
+    )
+    (property "Datasheet" "" (at 193.04 148.59 0)
+      (effects (font (size 1.27 1.27)) hide)
+    )
+    (pin "1")
+    (instances
+      (project "STM32F1-DevBoard"
+        (path "/978e1817-ddd6-4f04-b9a6-ae7fae5b1d1d"
+          (reference "#PWR04") (unit 1)
+        )
+      )

Commit message: Add files via upload
Changed lines of the file:
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@@
   (junction (at 157.48 66.04) (diameter 0) (color 0 0 0 0)
+  )
+  (junction (at 53.34 95.25) (diameter 0) (color 0 0 0 0)
   )
   (junction (at 195.58 73.66) (diameter 0) (color 0 0 0 0)
@@
     (stroke (width 0) (type default))
   )
-  (wire (pts (xy 45.72 101.6) (xy 45.72 102.87))
+  (wire (pts (xy 45.72 95.25) (xy 45.72 102.87))
     (stroke (width 0) (type default))
   )
@@
   )
   (wire (pts (xy 213.36 49.53) (xy 210.82 49.53))
+    (stroke (width 0) (type default))
+  )
+  (wire (pts (xy 45.72 95.25) (xy 53.34 95.25))
     (stroke (width 0) (type default))
   )
@@
     )
   )
-  (symbol (lib_id "power:+3.3V") (at 45.72 101.6 0) (unit 1)
-    (in_bom yes) (on_board yes) (dnp no)
-    (property "Reference" "#PWR0106" (at 45.72 105.41 0)
-      (effects (font (size 1.27 1.27)) hide)
-    )
-    (property "Value" "+3.3V" (at 45.72 95.25 90)
-      (effects (font (size 1.27 1.27)))
-    )
-    (property "Footprint" "" (at 45.72 101.6 0)
-      (effects (font (size 1.27 1.27)) hide)
-    )
-    (property "Datasheet" "" (at 45.72 101.6 0)
-      (effects (font (size 1.27 1.27)) hide)
-    )
-    (pin "1")
-    (instances
-      (project "STM32F1-DevBoard"
-        (path "/978e1817-ddd6-4f04-b9a6-ae7fae5b1d1d"
-          (reference "#PWR0106") (unit 1)
-        )
-      )
-    )
-  )
