File: STM32F1-DevBoard.kicad_pcb (KiCad board)
At the start: 2 copper layers, 20.3 x 50.8 mm, 30 parts, among them SW1 SW_Push, SW2 SW_Push, U1 STM32F103C8T6, U2 AMS1117-3.3

Commit message: Add files via upload
Parts:
- added C6: 100nF, Capacitor_SMD:C_0603_1608Metric, B.Cu at (137.2, 106.7)
- added U3: W25Q32JVSS, Package_SO:SOIC-8_5.23x5.23mm_P1.27mm, B.Cu at (137.2, 101.6)
Connections:
- CH1 pad 20: +5V -> VBUS
Routing:
- net +5V: track 47.2 -> 4.58 mm, vias 1 -> 0
- net VBUS: track 38.3 -> 58.6 mm
- net NRST: track 48.0 -> 32.1 mm, vias 2 -> 0
- net GND: track 137.7 -> 123.3 mm, vias 9 -> 18
- net PA4: track 10.9 -> 25.1 mm
- net PD1: track 26.2 -> 38.8 mm
- net PD0: track 25.6 -> 35.4 mm, vias 0 -> 4
- net PA6: track 7.82 -> 15.7 mm, vias 0 -> 1
- net BOOT0: track 29.0 -> 36.5 mm
- net PA0: track 23.5 -> 16.8 mm, vias 1 -> 0
- net PB9: track 28.4 -> 23.1 mm
- net PA7: track 6.70 -> 12.0 mm
- net +3.3V: track 114.3 -> 110.9 mm, vias 6 -> 2
- net PA10: track 34.2 -> 31.1 mm, vias 2 -> 1
- net PC13: track 22.7 -> 24.7 mm
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Other:
- board text added: "VBUS"

Commit message: Add files via upload
Routing:
- net BOOT0: track 36.5 -> 37.9 mm
- net NRST: track 32.1 -> 33.3 mm
- net +3.3V: track 110.9 -> 111.9 mm

Commit message: Add files via upload
Connections:
- CH1 pad 20: VBUS -> +5V
- D4 pad 2: VBUS -> +3.3V
- UART1 pad 4: VBUS -> +5V
Routing:
- net VBUS: track 58.6 -> 0.00 mm, vias 2 -> 0
- net +5V: track 4.58 -> 59.9 mm, vias 0 -> 2
- net +3.3V: track 111.9 -> 118.3 mm
Other:
- board text removed: "VBUS"

Commit message: Add files via upload
Routing:
- net PD0: track 35.4 -> 36.9 mm
- net +3.3V: track 118.3 -> 117.3 mm

Commit message: Add files via upload
Parts:
- moved C1 0.25 mm to (140.2, 78.0)
- moved C2 0.25 mm to (134.1, 78.0)
- moved C3 0.25 mm to (142.2, 78.0)
- moved C4 0.25 mm to (132.1, 78.0)
- moved XTAL1 0.25 mm to (137.2, 78.0)
Routing:
- net BOOT0: track 37.9 -> 39.5 mm
- net +5V: track 59.9 -> 59.2 mm
- net GND: track 123.7 -> 123.2 mm

Commit message: Add files via upload
Other:
- board text added: "FLASH"
- board text added: "STM32F103C8T6 Development Board"
Changed lines of the file:
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@@
   (gr_rect (start 127 76.2) (end 147.32 127)
     (stroke (width 0.1) (type solid)) (fill none) (layer "Edge.Cuts"))
+  (gr_text "FLASH" (at 137.16 101.6) (layer "B.SilkS")
+    (effects (font (size 1 1) (thickness 0.15)) (justify mirror))
+  )
   (gr_text "5V" (at 131.445 122.555) (layer "B.SilkS")
     (effects (font (size 0.8 0.8) (thickness 0.15)) (justify mirror))
+  )
+  (gr_text "STM32F103C8T6\nDevelopment Board" (at 137.16 81.915) (layer "B.SilkS")
+    (effects (font (size 1 1) (thickness 0.15)) (justify mirror))
   )
   (gr_text "VBAT" (at 142.875 122.555) (layer "B.SilkS")
@@
   )
   (gr_text "NRST" (at 134.112 113.919) (layer "F.SilkS")
-    (effects (font (size 1 1) (thickness 0.2)))
+    (effects (font (size 1 1) (thickness 0.15)))
   )
   (gr_text "B15" (at 145.161 115.57 90) (layer "F.SilkS")
@@
   )
   (gr_text "PB2" (at 133.096 108.077) (layer "F.SilkS")
-    (effects (font (size 1 1) (thickness 0.2)))
+    (effects (font (size 1 1) (thickness 0.15)))
   )
   (gr_text "A5" (at 129.159 97.79 -90) (layer "F.SilkS")
@@
   )
   (gr_text "BOOT0" (at 140.208 113.919) (layer "F.SilkS")
-    (effects (font (size 1 1) (thickness 0.2)))
+    (effects (font (size 1 1) (thickness 0.15)))
   )
   (gr_text "RST" (at 129.159 118.11 -90) (layer "F.SilkS")
@@
   )
   (gr_text "PWR" (at 141.224 108.077) (layer "F.SilkS")
-    (effects (font (size 1 1) (thickness 0.2)))
+    (effects (font (size 1 1) (thickness 0.15)))
   )
   (gr_text "C13" (at 129.159 77.47 -90) (layer "F.SilkS")

Commit message: Add files via upload
Routing:
- net PD0: track 36.7 -> 35.4 mm
Changed lines of the file:
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@@
   (segment (start 130.175 93.1972) (end 132.7558 95.778) (width 0.25) (layer "B.Cu") (net 7))
   (segment (start 130.175 84.455) (end 130.175 93.1972) (width 0.25) (layer "B.Cu") (net 7))
-  (segment (start 144.402485 99.106615) (end 142.036 101.4731) (width 0.25) (layer "F.Cu") (net 8))
+  (segment (start 139.704 101.4731) (end 137.795 99.5641) (width 0.25) (layer "F.Cu") (net 8))
   (segment (start 140.9398 83.5333) (end 140.9398 90.9329) (width 0.25) (layer "F.Cu") (net 8))
+  (segment (start 144.371196 99.137904) (end 142.036 101.4731) (width 0.25) (layer "F.Cu") (net 8))
   (segment (start 135.5056 98.8849) (end 134.747 98.1263) (width 0.25) (layer "F.Cu") (net 8))
   (segment (start 142.72 77.978) (end 142.72 79.2029) (width 0.25) (layer "F.Cu") (net 8))
+  (segment (start 144.448405 99.137904) (end 144.371196 99.137904) (width 0.25) (layer "F.Cu") (net 8))
   (segment (start 142.72 79.2029) (end 141.41 80.5129) (width 0.25) (layer "F.Cu") (net 8))
   (segment (start 141.41 83.0631) (end 140.9398 83.5333) (width 0.25) (layer "F.Cu") (net 8))
   (segment (start 141.41 81.788) (end 141.41 83.0631) (width 0.25) (layer "F.Cu") (net 8))
   (segment (start 142.036 101.4731) (end 139.704 101.4731) (width 0.25) (layer "F.Cu") (net 8))
-  (segment (start 139.704 101.4731) (end 137.795 99.5641) (width 0.25) (layer "F.Cu") (net 8))
-  (segment (start 145.370342 99.106615) (end 144.402485 99.106615) (width 0.25) (layer "F.Cu") (net 8))
   (segment (start 135.846 98.8849) (end 135.5056 98.8849) (width 0.25) (layer "F.Cu") (net 8))
   (segment (start 141.41 80.5129) (end 141.41 81.788) (width 0.25) (layer "F.Cu") (net 8))
-  (via (at 145.370342 99.106615) (size 0.8) (drill 0.4) (layers "F.Cu" "B.Cu") (net 8))
+  (via (at 144.448405 99.137904) (size 0.8) (drill 0.4) (layers "F.Cu" "B.Cu") (net 8))
   (via (at 135.846 98.8849) (size 0.8) (drill 0.4) (layers "F.Cu" "B.Cu") (net 8))
   (via (at 137.795 99.5641) (size 0.8) (drill 0.4) (layers "F.Cu" "B.Cu") (net 8))
@@
   (segment (start 144.2305 94.2236) (end 140.9398 90.9329) (width 0.25) (layer "B.Cu") (net 8))
   (segment (start 136.5252 99.5641) (end 135.846 98.8849) (width 0.25) (layer "B.Cu") (net 8))
-  (segment (start 144.2305 97.966773) (end 144.2305 94.2236) (width 0.25) (layer "B.Cu") (net 8))
-  (segment (start 145.370342 99.106615) (end 144.2305 97.966773) (width 0.25) (layer "B.Cu") (net 8))
+  (segment (start 144.448405 99.137904) (end 144.2305 98.919999) (width 0.25) (layer "B.Cu") (net 8))
   (segment (start 137.795 99.5641) (end 136.5252 99.5641) (width 0.25) (layer "B.Cu") (net 8))
+  (segment (start 144.2305 98.919999) (end 144.2305 94.2236) (width 0.25) (layer "B.Cu") (net 8))
   (segment (start 132.91 79.2597) (end 131.6283 77.978) (width 0.25) (layer "F.Cu") (net 9))
   (segment (start 136.260306 100.346806) (end 134.3934 98.4799) (width 0.25) (layer "F.Cu") (net 9))
