File: STM32F1-DevBoard.kicad_pcb (KiCad board)
At the start: 2 copper layers, 20.3 x 50.8 mm, 32 parts, among them SW1 SW_Push, SW2 SW_Push, U1 STM32F103C8T6, U2 AMS1117-3.3, U3 W25Q32JVSS

Commit message: Add files via upload
Parts:
- LED1: renamed from D1; value 19-217/BHC-ZL1M2RY/3T -> 19-217/GHC-YR1S2/3T
- LED2: renamed from D2; value 19-217/GHC-YR1S2/3T -> KT-0603R
Routing:
- net BOOT0: track 39.5 -> 38.5 mm
- net VB: track 42.1 -> 41.5 mm

Commit message: Add files via upload
Parts:
- removed D4: 1N5819WS, Diode_SMD:D_SOD-323
- removed UART1: Conn_01x06, Connector_PinHeader_2.54mm:PinHeader_1x06_P2.54mm_Horizontal
- added D1: 1N5819WS, Diode_SMD:D_SOD-323, F.Cu at (141.6, 104.8)
- added H1: MountingHole, MountingHole:MountingHole_2.2mm_M2, F.Cu at (130.8, 125.7)
- added H2: MountingHole, MountingHole:MountingHole_2.2mm_M2, F.Cu at (130.8, 77.5)
- added H3: MountingHole, MountingHole:MountingHole_2.2mm_M2, F.Cu at (143.5, 77.5)
- added H4: MountingHole, MountingHole:MountingHole_2.2mm_M2, F.Cu at (143.5, 125.7)
- added J1: USB_C_Receptacle_USB2.0, Connector_USB:USB_C_Receptacle_XKB_U262-16XN-4BVC11, F.Cu at (137.2, 122.8)
- added R3: 5.1kΩ, Resistor_SMD:R_0402_1005Metric, F.Cu at (131.1, 122.6)
- added R6: 5.1kΩ, Resistor_SMD:R_0402_1005Metric, F.Cu at (143.3, 122.6)
- added R7: 1.5kΩ, Resistor_SMD:R_0402_1005Metric, F.Cu at (137.2, 108.6)
- C1, C2: value 15pF -> 10pF
- C11: value 1μF -> 10uF
- C12: value 100μF -> 10uF; footprint Capacitor_SMD:C_1206_3216Metric -> Capacitor_SMD:C_0402_1005Metric
- C3, C4: value 30pF -> 20pF
- C6: footprint Capacitor_SMD:C_0603_1608Metric -> Capacitor_SMD:C_0603_1608Metric_Pad1.08x0.95mm_HandSolder
- R1, R2, R4, R5: value 10KΩ -> 10kΩ
- XTAL2: footprint Crystal:Crystal_SMD_HC49-SD -> Crystal:Crystal_SMD_5032-2Pin_5.0x3.2mm
- moved R4 32.4 mm to (135.9, 79.4)
- moved R5 32.4 mm to (138.4, 79.4)
- moved LED1 30.5 mm to (133.3, 79.4)
- moved LED2 30.5 mm to (141.0, 79.4)
- moved C11 19.6 mm to (137.2, 107.3), turned to 0 degrees
- moved C10 16.6 mm to (137.2, 80.6)
- moved C7 16.4 mm to (141.6, 101.3), turned to 0 degrees
- moved C8 16.4 mm to (141.6, 100.2), turned to 0 degrees
- moved C9 16.4 mm to (141.6, 102.5), turned to 0 degrees
- moved U2 15.1 mm to (135.9, 102.9)
- moved D3 12.2 mm to (140.3, 81.9)
- moved C5 12.1 mm to (137.2, 81.9), turned to 0 degrees
- moved C12 11.3 mm to (141.6, 99.1)
- moved C3 11.2 mm to (136.4, 87.5), turned to 180 degrees
- moved C2 10.5 mm to (138.4, 87.5), turned to 180 degrees
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Connections:
- C11 pad 1: +5V -> VCC
- C2 pad 1: GND -> PC15
- C2 pad 2: PC15 -> GND
- C4 pad 1: GND -> PD1
- C4 pad 2: PD1 -> GND
- U2 pad 3: +5V -> VCC
Routing:
- net +5V: track 59.2 -> 0.00 mm, vias 2 -> 0
- net PA11: track 5.99 -> 46.8 mm, vias 0 -> 2
- net GND: track 123.2 -> 163.9 mm, vias 18 -> 15
- net PA12: track 5.94 -> 38.7 mm, vias 0 -> 3
- net PD1: track 38.6 -> 7.91 mm, vias 2 -> 0
- net PD0: track 35.4 -> 6.66 mm, vias 4 -> 0
- net PB2: track 12.0 -> 40.7 mm, vias 0 -> 3
- net VBUS: track 0.00 -> 25.2 mm, vias 0 -> 2
- net PB13: track 18.6 -> 38.9 mm, vias 0 -> 2
- net PA10: track 30.7 -> 14.4 mm
- net NRST: track 33.3 -> 47.3 mm, vias 0 -> 1
- net VCC: track 0.00 -> 11.3 mm
- net PB10: track 10.4 -> 21.1 mm
- net PC14: track 33.9 -> 23.4 mm
- net PC15: track 29.9 -> 20.1 mm
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Other:
- board text added: "VB"
- board text removed: "G"
- board text removed: "NC"
- board text removed: "RX"
- board text removed: "TX"
- board text removed: "VBAT"

Commit message: Add files via upload
Parts:
- moved J1 1.08 mm to (137.2, 123.8)
Routing:
- net PA12: track 38.7 -> 40.8 mm
- net GND: track 163.9 -> 165.5 mm
- net VBUS: track 25.2 -> 26.8 mm
- net Net-(J1-CC2): track 7.27 -> 6.20 mm
- net Net-(J1-CC1): track 7.40 -> 6.53 mm

Commit message: Add files via upload
Parts:
- moved C13 0.64 mm to (134.0, 108.0)
- moved R2 0.64 mm to (140.3, 108.0)
- moved SW2 0.63 mm to (140.3, 114.3)
- moved SW1 0.61 mm to (134.0, 114.3)
Connections:
- CH1 pad 20: +5V -> VBUS
Routing:
- net VBUS: track 26.8 -> 37.0 mm
- net PA11: track 47.0 -> 38.5 mm, vias 2 -> 4
- net GND: track 165.5 -> 170.4 mm
- net PB14: track 24.4 -> 28.5 mm
- net PB12: track 29.9 -> 33.9 mm
- net PA12: track 40.8 -> 38.9 mm, vias 3 -> 4
- net +3.3V: track 114.4 -> 116.0 mm
- net BOOT0: track 30.2 -> 31.4 mm
- net Net-(J1-CC2): track 6.20 -> 5.66 mm

Commit message: Add files via upload
Routing:
- net PA12: track 38.9 -> 40.8 mm

Commit message: Add files via upload
Connections:
- CH1 pad 20: VBUS -> VCC
Routing:
- net VCC: track 11.3 -> 34.2 mm
- net VBUS: track 36.8 -> 24.4 mm
- net GND: track 170.4 -> 162.5 mm, vias 15 -> 14
- net NRST: track 47.0 -> 50.9 mm, vias 1 -> 2
- net PB2: track 40.7 -> 41.2 mm

Commit message: Add files via upload
Other:
- board text removed: "STM32F103C8T6 Development Board"
Changed lines of the file:
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@@
-    (effects (font (size 1 1) (thickness 0.2) bold) (justify mirror))
-  )
-  (gr_text "STM32F103C8T6\nDevelopment Board" (at 137.16 80.01) (layer "B.SilkS")
     (effects (font (size 1 1) (thickness 0.2) bold) (justify mirror))
   )
@@
   (segment (start 144.3729 107.95) (end 146.05 107.95) (width 0.25) (layer "B.Cu") (net 2))
   (segment (start 137.367228 100.109301) (end 137.367228 100.240228) (width 0.25) (layer "B.Cu") (net 2))
+  (segment (start 141.196 88.6989) (end 141.196 87.503) (width 0.5) (layer "F.Cu") (net 3))
   (segment (start 132.74 100.57) (end 132.115 101.195) (width 0.25) (layer "F.Cu") (net 3))
   (segment (start 139.41 96.484) (end 139.41 98.1425) (width 0.25) (layer "F.Cu") (net 3))
@@
   (segment (start 137.287 83.439) (end 137.287 84.709) (width 0.5) (layer "F.Cu") (net 3))
   (segment (start 137.64 79.655) (end 137.64 80.645) (width 0.25) (layer "F.Cu") (net 3))
-  (segment (start 141.097 88.7979) (end 141.097 87.602) (width 0.25) (layer "F.Cu") (net 3))
   (segment (start 142.4795 91.3086) (end 142.4795 90.4669) (width 0.25) (layer "F.Cu") (net 3))
   (segment (start 139.2074 95.7426) (end 139.2074 93.2613) (width 0.25) (layer "F.Cu") (net 3))
@@
   (segment (start 141.7742 104.4071) (end 141.5611 104.4071) (width 0.25) (layer "F.Cu") (net 3))
   (segment (start 131.4631 106.1931) (end 131.4631 101.8469) (width 0.25) (layer "F.Cu") (net 3))
-  (segment (start 140.8845 89.0104) (end 141.097 88.7979) (width 0.25) (layer "F.Cu") (net 3))
   (segment (start 139.065 107.95) (end 138.43 107.315) (width 0.25) (layer "F.Cu") (net 3))
   (segment (start 131.4631 101.8469) (end 132.74 100.57) (width 0.25) (layer "F.Cu") (net 3))
   (segment (start 132.115 101.195) (end 131.9699 101.195) (width 0.25) (layer "F.Cu") (net 3))
-  (segment (start 141.097 87.602) (end 141.196 87.503) (width 0.25) (layer "F.Cu") (net 3))
   (segment (start 139.825 107.95) (end 139.065 107.95) (width 0.25) (layer "F.Cu") (net 3))
   (segment (start 141.3225 91.73) (end 142.0581 91.73) (width 0.25) (layer "F.Cu") (net 3))
@@
   (segment (start 136.6117 82.9897) (end 136.779 83.058) (width 0.5) (layer "F.Cu") (net 3))
   (segment (start 132.300181 87.407893) (end 131.829893 87.407893) (width 0.5) (layer "F.Cu") (net 3))
+  (segment (start 140.8845 89.0104) (end 141.196 88.6989) (width 0.5) (layer "F.Cu") (net 3))
   (segment (start 131.9699 101.195) (end 131.9699 96.5022) (width 0.25) (layer "F.Cu") (net 3))
   (segment (start 137.287 86.84) (end 137.287 87.094) (width 0.5) (layer "F.Cu") (net 3))
@@
   (segment (start 128.27 95.1715) (end 128.27 95.25) (width 0.25) (layer "F.Cu") (net 18))
   (segment (start 132.9975 91.73) (end 131.7115 91.73) (width 0.25) (layer "F.Cu") (net 18))
-  (segment (start 133.429983 91.1355) (end 135.2817 91.1355) (width 0.25) (layer "B.Cu") (net 18))
-  (segment (start 136.1656 92.0194) (end 140.7044 92.0194) (width 0.25) (layer "B.Cu") (net 18))
+  (segment (start 130.848289 88.553806) (end 133.429983 91.1355) (width 0.25) (layer "B.Cu") (net 18))
   (segment (start 135.2817 91.1355) (end 136.1656 92.0194) (width 0.25) (layer "B.Cu") (net 18))
-  (segment (start 140.7044 92.0194) (end 140.76 92.075) (width 0.25) (layer "B.Cu") (net 18))
   (segment (start 128.27 95.25) (end 129.6695 93.8505) (width 0.25) (layer "B.Cu") (net 18))
+  (segment (start 129.6695 93.8505) (end 129.6695 89.173405) (width 0.25) (layer "B.Cu") (net 18))
   (segment (start 130.289099 88.553806) (end 130.848289 88.553806) (width 0.25) (layer "B.Cu") (net 18))
   (segment (start 129.6695 89.173405) (end 130.289099 88.553806) (width 0.25) (layer "B.Cu") (net 18))
-  (segment (start 130.848289 88.553806) (end 133.429983 91.1355) (width 0.25) (layer "B.Cu") (net 18))
-  (segment (start 129.6695 93.8505) (end 129.6695 89.173405) (width 0.25) (layer "B.Cu") (net 18))
+  (segment (start 140.7044 92.0194) (end 140.76 92.075) (width 0.25) (layer "B.Cu") (net 18))
+  (segment (start 136.1656 92.0194) (end 140.7044 92.0194) (width 0.25) (layer "B.Cu") (net 18))
+  (segment (start 133.429983 91.1355) (end 135.2817 91.1355) (width 0.25) (layer "B.Cu") (net 18))
   (segment (start 129.3969 94.613) (end 129.3969 96.6631) (width 0.25) (layer "F.Cu") (net 19))
   (segment (start 131.7799 92.23) (end 129.3969 94.613) (width 0.25) (layer "F.Cu") (net 19))

Commit message: Add files via upload
Parts:
- moved H1 0.38 mm to (131.2, 125.7)
- moved H2 0.38 mm to (131.2, 77.5)
- moved H3 0.38 mm to (143.1, 77.5)
- moved H4 0.38 mm to (143.1, 125.7)
- moved R3 0.38 mm to (131.4, 122.6)
- moved R6 0.38 mm to (142.9, 122.6)
