File: STM32F1-DevBoard.kicad_pcb (KiCad board)
At the start: 2 copper layers, 20.3 x 50.8 mm, 39 parts, among them J1 USB_C_Receptacle_USB2.0, SW1 SW_Push, SW2 SW_Push, U1 STM32F103C8T6, U2 AMS1117-3.3, U3 W25Q32JVSS

Commit message: Add files via upload
Parts:
- moved H1 0.13 mm to (131.3, 125.7)
- moved H2 0.13 mm to (131.3, 77.5)
- moved H3 0.13 mm to (143.0, 77.5)
- moved H4 0.13 mm to (143.0, 125.7)
Changed lines of the file:
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@@
   )
   (footprint "MountingHole:MountingHole_2.2mm_M2" (layer "F.Cu")
-    (at 131.191 77.47)
+    (at 131.318 77.47)
     (descr "Mounting Hole 2.2mm, no annular, M2")
     (tags "mounting hole 2.2mm no annular m2")
@@
   )
   (footprint "MountingHole:MountingHole_2.2mm_M2" (layer "F.Cu")
-    (at 143.129 77.47)
+    (at 143.002 77.47)
     (descr "Mounting Hole 2.2mm, no annular, M2")
     (tags "mounting hole 2.2mm no annular m2")
@@
   )
   (footprint "MountingHole:MountingHole_2.2mm_M2" (layer "F.Cu")
-    (at 143.129 125.73)
+    (at 143.002 125.73)
     (descr "Mounting Hole 2.2mm, no annular, M2")
     (tags "mounting hole 2.2mm no annular m2")
@@
   )
   (footprint "MountingHole:MountingHole_2.2mm_M2" (layer "F.Cu")
-    (at 131.191 125.73)
+    (at 131.318 125.73)
     (descr "Mounting Hole 2.2mm, no annular, M2")
     (tags "mounting hole 2.2mm no annular m2")

Commit message: Add files via upload
Parts:
- moved R6 0.13 mm to (143.0, 122.6)
- moved R3 0.13 mm to (131.3, 122.6)
Other:
- board text added: "SOIC-8"
- board text removed: "FLASH"
Changed lines of the file:
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@@
   )
   (footprint "Resistor_SMD:R_0402_1005Metric" (layer "F.Cu")
-    (at 142.875 122.555 90)
+    (at 143.002 122.555 90)
     (descr "Resistor SMD 0402 (1005 Metric), square (rectangular) end terminal, IPC_7351 nominal, (Body size source: IPC-SM-782 page 72, https://www.pcb-3d.com/wordpress/wp-content/uploads/ipc-sm-782a_amendment_1_and_2.pdf), generated with kicad-footprint-generator")
     (tags "resistor")
@@
   )
   (footprint "Resistor_SMD:R_0402_1005Metric" (layer "F.Cu")
-    (at 131.445 122.555 90)
+    (at 131.318 122.555 90)
     (descr "Resistor SMD 0402 (1005 Metric), square (rectangular) end terminal, IPC_7351 nominal, (Body size source: IPC-SM-782 page 72, https://www.pcb-3d.com/wordpress/wp-content/uploads/ipc-sm-782a_amendment_1_and_2.pdf), generated with kicad-footprint-generator")
     (tags "resistor")
@@
     )
   )
-  (gr_line (start 127.635 106.68) (end 128.905 106.68)
-    (stroke (width 0.15) (type default)) (layer "B.SilkS"))
-  (gr_line (start 145.415 96.52) (end 146.685 96.52)
-    (stroke (width 0.15) (type default)) (layer "B.SilkS"))
-  (gr_line (start 127.635 86.36) (end 128.905 86.36)
-    (stroke (width 0.15) (type default)) (layer "B.SilkS"))
-  (gr_line (start 127.635 116.84) (end 128.905 116.84)
-    (stroke (width 0.15) (type default)) (layer "B.SilkS"))
-  (gr_line (start 127.635 96.52) (end 128.905 96.52)
-    (stroke (width 0.15) (type default)) (layer "B.SilkS"))
-  (gr_line (start 145.415 86.36) (end 146.685 86.36)
-    (stroke (width 0.15) (type default)) (layer "B.SilkS"))
-  (gr_line (start 145.415 116.84) (end 146.685 116.84)
-    (stroke (width 0.15) (type default)) (layer "B.SilkS"))
-  (gr_line (start 145.415 106.68) (end 146.685 106.68)
-    (stroke (width 0.15) (type default)) (layer "B.SilkS"))
   (gr_line (start 145.415 116.84) (end 146.685 116.84)
     (stroke (width 0.15) (type default)) (layer "F.SilkS"))
@@
     (effects (font (size 0.8 0.8) (thickness 0.15)) (justify bottom mirror))
   )
-  (gr_text "FLASH" (at 137.16 93.98) (layer "B.SilkS")
-    (effects (font (size 1 1) (thickness 0.2) bold) (justify mirror))
+  (gr_text "SOIC-8" (at 137.16 93.98) (layer "B.SilkS")
+    (effects (font (size 0.8 0.8) (thickness 0.15) bold) (justify mirror))
   )
   (gr_text "RST" (at 129.54 118.11 -90) (layer "B.SilkS")
@@
     (format (prefix "") (suffix "") (units 3) (units_format 1) (precision 2))
     (style (thickness 0.15) (arrow_length 1.27) (text_position_mode 0) (extension_height 0.58642) (extension_offset 0.5) keep_text_aligned)
+  )
+  (dimension (type aligned) (layer "Cmts.User")
+    (pts (xy 128.27 125.73) (xy 131.318 125.73))
+    (height 8.255)
+    (gr_text "3.048 mm" (at 129.794 135.89) (layer "Cmts.User")
+      (effects (font (size 1 1) (thickness 0.15)))
+    )
+    (format (prefix "") (suffix "") (units 3) (units_format 1) (precision 3))
+    (style (thickness 0.15) (arrow_length 1.27) (text_position_mode 2) (extension_height 0.58642) (extension_offset 0.5) keep_text_aligned)
+  )
+  (dimension (type aligned) (layer "Cmts.User")
+    (pts (xy 131.318 77.47) (xy 143.002 77.47))
+    (height -6.35)
+    (gr_text "11.684 mm" (at 137.16 69.97) (layer "Cmts.User")
+      (effects (font (size 1 1) (thickness 0.15)))
+    )
+    (format (prefix "") (suffix "") (units 3) (units_format 1) (precision 3))
+    (style (thickness 0.15) (arrow_length 1.27) (text_position_mode 0) (extension_height 0.58642) (extension_offset 0.5) keep_text_aligned)
+  )
+  (dimension (type aligned) (layer "Cmts.User")
+    (pts (xy 146.05 123.19) (xy 146.05 125.73))
+    (height -3.81)
+    (gr_text "2.540 mm" (at 151.765 124.46 90) (layer "Cmts.User")
+      (effects (font (size 1 1) (thickness 0.15)))
+    )
+    (format (prefix "") (suffix "") (units 3) (units_format 1) (precision 3))
+    (style (thickness 0.15) (arrow_length 1.27) (text_position_mode 2) (extension_height 0.58642) (extension_offset 0.5) keep_text_aligned)
   )
   (segment (start 143.7199 100.367885) (end 143.7199 99.2216) (width 0.25) (layer "F.Cu") (net 1))
@@
   (segment (start 142.4795 91.3086) (end 142.4795 90.4669) (width 0.25) (layer "F.Cu") (net 3))
   (segment (start 139.2074 95.7426) (end 139.2074 93.2613) (width 0.25) (layer "F.Cu") (net 3))
-  (segment (start 142.875 123.065) (end 142.875 123.505) (width 0.25) (layer "F.Cu") (net 3))
   (segment (start 136.41 91.0853) (end 136.3216 91.1737) (width 0.25) (layer "F.Cu") (net 3))
   (segment (start 130.556 86.36) (end 130.556 83.552) (width 0.5) (layer "F.Cu") (net 3))
@@
   (segment (start 141.5611 104.4071) (end 139.825 106.1432) (width 0.25) (layer "F.Cu") (net 3))
   (segment (start 133.0129 82.9897) (end 136.6117 82.9897) (width 0.5) (layer "F.Cu") (net 3))
+  (segment (start 143.002 123.065) (end 143.002 123.378) (width 0.25) (layer "F.Cu") (net 3))
   (segment (start 134.9227 117.45) (end 133.81 118.5627) (width 0.25) (layer "F.Cu") (net 3))
   (segment (start 133.245 120.72) (end 132.84 120.72) (width 0.25) (layer "F.Cu") (net 3))
   (segment (start 142.0581 91.73) (end 142.4795 91.3086) (width 0.25) (layer "F.Cu") (net 3))
   (segment (start 137.287 84.709) (end 137.287 86.84) (width 0.5) (layer "F.Cu") (net 3))
-  (segment (start 142.875 123.505) (end 141.48 124.9) (width 0.25) (layer "F.Cu") (net 3))
   (segment (start 135.841 79.934) (end 135.841 80.5124) (width 0.25) (layer "F.Cu") (net 3))
   (segment (start 135.89 117.45) (end 134.9227 117.45) (width 0.25) (layer "F.Cu") (net 3))
@@
   (segment (start 137.92 79.375) (end 137.64 79.655) (width 0.25) (layer "F.Cu") (net 3))
   (segment (start 142.085 99.06) (end 142.085 98.1907) (width 0.25) (layer "F.Cu") (net 3))
+  (segment (start 143.002 123.378) (end 141.48 124.9) (width 0.25) (layer "F.Cu") (net 3))
   (segment (start 141.427352 84.328) (end 139.573 84.328) (width 0.5) (layer "F.Cu") (net 3))
   (segment (start 141.859 84.759648) (end 141.427352 84.328) (width 0.5) (layer "F.Cu") (net 3))
   (segment (start 142.1073 102.5113) (end 142.1073 104.074) (width 0.25) (layer "F.Cu") (net 3))
+  (segment (start 131.318 123.378) (end 132.84 124.9) (width 0.25) (layer "F.Cu") (net 3))
   (segment (start 142.085 101.346) (end 142.085 102.489) (width 0.25) (layer "F.Cu") (net 3))
   (segment (start 140.51 120.155) (end 140.51 120.245) (width 0.25) (layer "F.Cu") (net 3))
@@
   (segment (start 131.1183 82.9897) (end 133.0129 82.9897) (width 0.5) (layer "F.Cu") (net 3))
   (segment (start 131.9699 96.5022) (end 132.2421 96.23) (width 0.25) (layer "F.Cu") (net 3))
-  (segment (start 131.445 123.505) (end 132.84 124.9) (width 0.25) (layer "F.Cu") (net 3))
   (segment (start 142.085 102.489) (end 142.1073 102.5113) (width 0.25) (layer "F.Cu") (net 3))
   (segment (start 141.196 87.503) (end 141.859 86.84) (width 0.5) (layer "F.Cu") (net 3))
@@
   (segment (start 139.573 84.328) (end 137.668 84.328) (width 0.5) (layer "F.Cu") (net 3))
   (segment (start 141.7742 104.4071) (end 141.5611 104.4071) (width 0.25) (layer "F.Cu") (net 3))
+  (segment (start 131.318 123.065) (end 131.318 123.378) (width 0.25) (layer "F.Cu") (net 3))
   (segment (start 139.065 107.95) (end 138.43 107.315) (width 0.25) (layer "F.Cu") (net 3))
   (segment (start 132.115 101.195) (end 131.9699 101.195) (width 0.25) (layer "F.Cu") (net 3))
@@
   (segment (start 132.300181 87.407893) (end 131.829893 87.407893) (width 0.5) (layer "F.Cu") (net 3))
   (segment (start 140.8845 89.0104) (end 141.196 88.6989) (width 0.5) (layer "F.Cu") (net 3))
-  (segment (start 131.445 123.065) (end 131.445 123.505) (width 0.25) (layer "F.Cu") (net 3))
   (segment (start 131.9699 101.195) (end 131.9699 96.5022) (width 0.25) (layer "F.Cu") (net 3))
   (segment (start 137.287 86.84) (end 137.287 87.094) (width 0.5) (layer "F.Cu") (net 3))
@@
   (segment (start 139.5485 116.205) (end 140.6408 117.2973) (width 0.25) (layer "B.Cu") (net 48))
   (segment (start 134.62 118.11) (end 136.525 116.205) (width 0.25) (layer "B.Cu") (net 48))
+  (segment (start 135.91 120.155) (end 135.91 120.98) (width 0.25) (layer "F.Cu") (net 49))
   (segment (start 135.91 120.98) (end 134.845 122.045) (width 0.25) (layer "F.Cu") (net 49))
-  (segment (start 134.845 122.045) (end 131.445 122.045) (width 0.25) (layer "F.Cu") (net 49))
-  (segment (start 135.91 120.155) (end 135.91 120.98) (width 0.25) (layer "F.Cu") (net 49))
+  (segment (start 134.845 122.045) (end 131.318 122.045) (width 0.25) (layer "F.Cu") (net 49))
   (segment (start 138.91 120.155) (end 138.91 121.069949) (width 0.25) (layer "F.Cu") (net 50))
-  (segment (start 139.885051 122.045) (end 142.875 122.045) (width 0.25) (layer "F.Cu") (net 50))
   (segment (start 138.91 121.069949) (end 139.885051 122.045) (width 0.25) (layer "F.Cu") (net 50))
+  (segment (start 139.885051 122.045) (end 143.002 122.045) (width 0.25) (layer "F.Cu") (net 50))
   (zone (net 0) (net_name "") (layer "F.Cu") (hatch edge 0.5)
     (connect_pads (clearance 0))
@@
     (polygon
       (pts
-        (xy 120.65 69.85)
-        (xy 120.65 133.35)
-        (xy 152.4 133.35)
-        (xy 152.4 69.85)
+        (xy 114.3 63.5)
+        (xy 114.3 139.7)
+        (xy 158.75 139.7)
+        (xy 158.75 63.5)
       )
     )

Commit message: Add files via upload
Routing:
- net PA12: track 40.8 -> 39.6 mm

Commit message: Add files via upload
Parts:
- moved C13 0.51 mm to (134.5, 108.0)
- moved D1 0.38 mm to (141.6, 105.2)
Routing:
- net VBUS: track 24.4 -> 22.9 mm
- net PA12: track 39.6 -> 40.2 mm
- net PA11: track 38.5 -> 38.0 mm

Commit message: Add files via upload
Parts:
- C11, C12: value 10uF -> 22uF; footprint Capacitor_SMD:C_0402_1005Metric -> Capacitor_SMD:C_0805_2012Metric
- moved H1 17.8 mm to (131.4, 108.0)
- moved H4 17.8 mm to (142.9, 108.0)
- moved R1 16.9 mm to (131.3, 124.8), turned to -90 degrees
- moved C8 1.15 mm to (141.5, 101.3)
- moved C7 1.02 mm to (141.5, 102.4)
- moved R4 0.90 mm to (136.5, 78.7), turned to -90 degrees
- moved R5 0.90 mm to (137.8, 78.7), turned to -90 degrees
- moved C9 0.90 mm to (141.5, 103.4)
- moved R2 0.74 mm to (139.7, 107.6), turned to 90 degrees
- moved LED1 0.64 mm to (134.0, 79.4)
- moved R7 0.64 mm to (137.2, 109.2)
- moved LED2 0.63 mm to (140.3, 79.4)
- moved D1 0.40 mm to (141.5, 105.5)
- moved C12 0.38 mm to (142.0, 99.1), turned to 90 degrees
- moved C11 0.25 mm to (137.2, 107.6)
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Routing:
- net PB2: track 41.2 -> 60.2 mm, vias 3 -> 5
- net PB10: track 21.1 -> 27.0 mm
- net NRST: track 50.9 -> 54.4 mm
- net BOOT0: track 31.0 -> 33.7 mm, vias 0 -> 2
- net PA13: track 11.0 -> 12.9 mm
- net VCC: track 34.0 -> 35.8 mm
- net VB: track 51.0 -> 49.6 mm
- net PA11: track 38.0 -> 39.4 mm
- net +3.3V: track 117.0 -> 118.2 mm
- net Net-(LED2-K): track 1.24 -> 2.23 mm
- net Net-(LED1-K): track 1.24 -> 2.23 mm
- net PA12: track 40.2 -> 41.1 mm

Commit message: Add files via upload
Parts:
- moved R1 45.0 mm to (131.4, 79.9), turned to 90 degrees
- moved R3 0.63 mm to (131.3, 123.2)
- moved R6 0.63 mm to (143.0, 123.2)
Routing:
- net PB2: track 60.2 -> 37.6 mm, vias 5 -> 2
- net PB10: track 27.0 -> 21.1 mm
- net GND: track 161.2 -> 163.2 mm, vias 14 -> 15
- net NRST: track 54.4 -> 52.9 mm
- net VCC: track 35.8 -> 34.9 mm

Commit message: Add files via upload
Changed lines of the file:
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@@
     (descr "SMD Crystal FC-135 https://support.epson.biz/td/api/doc_check.php?dl=brief_FC-135R_en.pdf")
     (tags "SMD SMT Crystal")
-    (property "JLCPCB Rotation Offset" "-180")
+    (property "JLCPCB Rotation Offset" "0")
     (property "LCSC" "C32346")
     (property "Sheetfile" "STM32F1-DevBoard.kicad_sch")
@@
   )
   (gr_text "PB2" (at 133.985 78.105) (layer "F.SilkS")
-    (effects (font (size 0.8 0.8) (thickness 0.15) bold) (justify bottom))
+    (effects (font (size 1 1) (thickness 0.2) bold) (justify bottom))
   )
   (gr_text "A5" (at 129.54 97.79 -90) (layer "F.SilkS")
@@
   )
   (gr_text "PWR" (at 140.335 78.105) (layer "F.SilkS")
-    (effects (font (size 0.8 0.8) (thickness 0.15) bold) (justify bottom))
+    (effects (font (size 1 1) (thickness 0.2) bold) (justify bottom))
   )
   (gr_text "C13" (at 129.54 77.47 -90) (layer "F.SilkS")
